Commit message: Add READMEs

File: nedo3_description/urdf/rack_b.urdf.xacro (robot description, xacro)
@@ -5,5 +5,5 @@
         <origin rpy="0 0 0" xyz="0 0 0"/>
         <geometry>
-          <mesh filename="package://nedo3_description/meshes/rack_b.stl" scale="0.001 0.001 0.001"/>
+          <mesh filename="package://nedo3_description/meshes/visual/rack_b.stl" scale="0.001 0.001 0.001"/>
         </geometry>
         <material name="white">

File: nedo3_description/urdf/rack_t.urdf.xacro (robot description, xacro)
@@ -5,5 +5,5 @@
         <origin rpy="0 0 0" xyz="0 0 0"/>
         <geometry>
-          <mesh filename="package://nedo3_description/meshes/rack_t.stl" scale="0.001 0.001 0.001"/>
+          <mesh filename="package://nedo3_description/meshes/visual/rack_t.stl" scale="0.001 0.001 0.001"/>
         </geometry>
         <material name="white">
