Commit message: Add part boxes

File: nedo3_description/urdf/nedo3_demo.urdf.xacro (robot description, xacro)
@@ -67,131 +67,18 @@
     <origin xyz="0 0 ${rack_t_elevation}" rpy="0 0 0"/>
   </xacro:rack_t>
-  <!-- <!-\- Put boxes on shooters -\-> -->
-  <!-- <xacro:include filename="$(find nedo3_description)/scenes/urdf/put_boxes_on_shooters.urdf.xacro"/> -->
-  <!-- <xacro:property name="rack_b_props" -->
-  <!-- 		  value="${xacro.load_yaml('$(find nedo3_description -->
-  <!-- 			 )/config/showcase_rack_b_props.yaml')}"/> -->
-  <!-- <xacro:property name="showcase_params" -->
-  <!-- 		  value="${xacro.load_yaml('$(find nedo3_routines -->
-  <!-- 			 )/config/showcase.yaml')}"/> -->
-  <!-- <xacro:property name="boxes" -->
-  <!-- 		  value="${showcase_params['boxes']}"/> -->
-  <!-- <xacro:property name="part_props" -->
-  <!-- 		  value="${showcase_params['motion_parameters']}"/> -->
-  <!-- <xacro:property name="box_props" -->
-  <!-- 		  value="${xacro.load_yaml('$(find nedo3_description -->
-  <!-- 			 )/config/box_props.yaml')}"/> -->
-  <!-- Spawning boxes for all shooters is computationally very intensive
-       because of its high recursive nature. -->
-  <!-- <xacro:put_boxes_on_shooters rack_b_props="${rack_b_props}" -->
-  <!-- 			       part_props="${part_props}" -->
-  <!-- 			       box_props="${box_props}"/> -->
-  <!-- Spawn boxes for each shooter one by one, -->
-  <!-- <xacro:put_boxes_on_shooter rack_b_name="rack_b_A" -->
-  <!-- 			      rack_b_prop="${rack_b_props['rack_b_A']}" -->
-  <!-- 			      boxes="${boxes}" -->
-  <!-- 			      part_props="${part_props}" -->
-  <!-- 			      box_props="${box_props}"/> -->
-  <!-- <xacro:put_boxes_on_shooter rack_b_name="rack_b_B" -->
-  <!-- 			      rack_b_prop="${rack_b_props['rack_b_B']}" -->
-  <!-- 			      boxes="${boxes}" -->
-  <!-- 			      part_props="${part_props}" -->
-  <!-- 			      box_props="${box_props}"/> -->
-  <!-- <xacro:put_boxes_on_shooter rack_b_name="rack_b_C" -->
-  <!-- 			      rack_b_prop="${rack_b_props['rack_b_C']}" -->
-  <!-- 			      boxes="${boxes}" -->
-  <!-- 			      part_props="${part_props}" -->
-  <!-- 			      box_props="${box_props}"/> -->
-  <!-- <xacro:put_boxes_on_shooter rack_b_name="rack_b_D" -->
-  <!-- 			      rack_b_prop="${rack_b_props['rack_b_D']}" -->
-  <!-- 			      boxes="${boxes}" -->
-  <!-- 			      part_props="${part_props}" -->
-  <!-- 			      box_props="${box_props}"/> -->
-  <!-- <xacro:put_boxes_on_shooter rack_b_name="rack_b_E" -->
-  <!-- 			      rack_b_prop="${rack_b_props['rack_b_E']}" -->
-  <!-- 			      boxes="${boxes}" -->
-  <!-- 			      part_props="${part_props}" -->
-  <!-- 			      box_props="${box_props}"/> -->
-  <!-- <xacro:put_boxes_on_shooter rack_b_name="rack_b_F" -->
-  <!-- 			      rack_b_prop="${rack_b_props['rack_b_F']}" -->
-  <!-- 			      boxes="${boxes}" -->
-  <!-- 			      part_props="${part_props}" -->
-  <!-- 			      box_props="${box_props}"/> -->
-  <!-- <xacro:put_boxes_on_shooter rack_b_name="rack_b_G" -->
-  <!-- 			      rack_b_prop="${rack_b_props['rack_b_G']}" -->
-  <!-- 			      boxes="${boxes}" -->
-  <!-- 			      part_props="${part_props}" -->
-  <!-- 			      box_props="${box_props}"/> -->
-  <!-- <xacro:put_boxes_on_shooter rack_b_name="rack_b_H" -->
-  <!-- 			      rack_b_prop="${rack_b_props['rack_b_H']}" -->
-  <!-- 			      boxes="${boxes}" -->
-  <!-- 			      part_props="${part_props}" -->
-  <!-- 			      box_props="${box_props}"/> -->
-  <!-- <xacro:put_boxes_on_shooter rack_b_name="rack_b_I" -->
-  <!-- 			      rack_b_prop="${rack_b_props['rack_b_I']}" -->
-  <!-- 			      boxes="${boxes}" -->
-  <!-- 			      part_props="${part_props}" -->
-  <!-- 			      box_props="${box_props}"/> -->
-  <!-- <xacro:put_boxes_on_shooter rack_b_name="rack_b_J" -->
-  <!-- 			      rack_b_prop="${rack_b_props['rack_b_J']}" -->
-  <!-- 			      boxes="${boxes}" -->
-  <!-- 			      part_props="${part_props}" -->
-  <!-- 			      box_props="${box_props}"/> -->
-  <!-- <!-\- Set staypoints for shooters -\-> -->
-  <!-- <xacro:include filename="$(find nedo3_description -->
-  <!-- 			   )/scenes/urdf/set_rack_b_staypoint.urdf.xacro"/> -->
-  <!-- <xacro:set_rack_b_staypoint rack_b_name="rack_b_A" -->
-  <!-- 			       rack_b_prop="${rack_b_props['rack_b_A']}" -->
-  <!-- 			       lane_width="${lane_width}"/> -->
-  <!-- <xacro:set_rack_b_staypoint rack_b_name="rack_b_B" -->
-  <!-- 			       rack_b_prop="${rack_b_props['rack_b_B']}" -->
-  <!-- 			       lane_width="${lane_width}"/> -->
-  <!-- <xacro:set_rack_b_staypoint rack_b_name="rack_b_C" -->
-  <!-- 			       rack_b_prop="${rack_b_props['rack_b_C']}" -->
-  <!-- 			       lane_width="${lane_width}"/> -->
-  <!-- <xacro:set_rack_b_staypoint rack_b_name="rack_b_F" -->
-  <!-- 			       rack_b_prop="${rack_b_props['rack_b_F']}" -->
-  <!-- 			       lane_width="${lane_width}"/> -->
-  <!-- <xacro:set_rack_b_staypoint rack_b_name="rack_b_H" -->
-  <!-- 			       rack_b_prop="${rack_b_props['rack_b_H']}" -->
-  <!-- 			       lane_width="${lane_width}"/> -->
-  <!-- <xacro:set_rack_b_staypoint rack_b_name="rack_b_J" -->
-  <!-- 			       rack_b_prop="${rack_b_props['rack_b_J']}" -->
-  <!-- 			       lane_width="${lane_width}"/> -->
-  <!-- <!-\- Set staypoints for boxes -\-> -->
-  <!-- <xacro:include filename="$(find nedo3_description -->
-  <!-- 			   )/scenes/urdf/set_box_staypoints.urdf.xacro"/> -->
-  <!-- <xacro:set_box_staypoints rack_b_name="rack_b_D" -->
-  <!-- 			    rack_b_prop="${rack_b_props['rack_b_D']}" -->
-  <!-- 			    part_props="${part_props}" -->
-  <!-- 			    box_props="${box_props}" -->
-  <!-- 			    lane_width="${lane_width}"/> -->
-  <!-- <xacro:set_box_staypoints rack_b_name="rack_b_E" -->
-  <!-- 			    rack_b_prop="${rack_b_props['rack_b_E']}" -->
-  <!-- 			    part_props="${part_props}" -->
-  <!-- 			    box_props="${box_props}" -->
-  <!-- 			    lane_width="${lane_width}"/> -->
-  <!-- <xacro:set_box_staypoints rack_b_name="rack_b_G" -->
-  <!-- 			    rack_b_prop="${rack_b_props['rack_b_G']}" -->
-  <!-- 			    part_props="${part_props}" -->
-  <!-- 			    box_props="${box_props}" -->
-  <!-- 			    lane_width="${lane_width}"/> -->
-  <!-- <xacro:set_box_staypoints rack_b_name="rack_b_I" -->
-  <!-- 			    rack_b_prop="${rack_b_props['rack_b_I']}" -->
-  <!-- 			    part_props="${part_props}" -->
-  <!-- 			    box_props="${box_props}" -->
-  <!-- 			    lane_width="${lane_width}"/> -->
-  <!-- <!-\- Set staypoints for home and charger -\-> -->
-  <!-- <xacro:include filename="$(find nedo3_description -->
-  <!-- 			   )/scenes/urdf/set_staypoint.urdf.xacro"/> -->
-  <!-- <xacro:set_staypoint suffix="_charger" parent="ground" -->
-  <!-- 		       x="7.250" y="${lane_separation/2}"/> -->
-  <!-- <xacro:set_staypoint suffix="_home" parent="ground" -->
-  <!-- 		       x="0.300" y="${-lane_separation/2}" theta="${pi}"/> -->
-  <!-- <!-\- Set staypoints for north-west and south-east -\-> -->
-  <!-- <xacro:set_staypoint suffix="_NW" parent="ground" -->
-  <!-- 		       x="${0.650 - 0.495 - 0.225}" y="${lane_separation/2}"/> -->
-  <!-- <xacro:set_staypoint suffix="_SE" parent="ground" -->
-  <!-- 		       x="${7.350 + 0.495 - 0.225}" y="${-lane_separation/2}" -->
-  <!-- 		       theta="${pi}"/> -->
+  <!-- Put boxes on shooters -->
+  <xacro:include filename="$(find nedo3_description
+			   )/urdf/put_boxes_on_racks.urdf.xacro"/>
+  <xacro:property name="rack_props"
+		  value="${xacro.load_yaml('$(find nedo3_description
+			 )/config/rack_props.yaml')}"/>
+  <xacro:property name="part_props"
+		  value="${xacro.load_yaml('$(find nedo3_description
+			 )/config/part_props.yaml')}"/>
+  <xacro:property name="box_props"
+		  value="${xacro.load_yaml('$(find nedo3_description
+			 )/config/box_props.yaml')}"/>
+  <xacro:put_boxes_on_racks rack_props="${rack_props}"
+			    part_props="${part_props}"
+			    box_props="${box_props}"/>
 </robot>

Commit message: Change elevetion and setback of rack_t

File: nedo3_description/urdf/nedo3_demo.urdf.xacro (robot description, xacro)
@@ -7,5 +7,6 @@
   <xacro:property name="rack_width"		value="0.85"/>
   <xacro:property name="rack_separation"	value="0.04"/>
-  <xacro:property name="rack_t_elevation"	value="0.20"/>
+  <xacro:property name="rack_t_setback"		value="-0.050"/>
+  <xacro:property name="rack_t_elevation"	value="0.595"/>
   <!-- Root frame -->
   <link name="world"/>
@@ -36,5 +37,5 @@
 			   )/urdf/rack_t.urdf.xacro"/>
   <xacro:rack_t name="rack_t0" parent="rack_b0">
-    <origin xyz="0 0 ${rack_t_elevation}" rpy="0 0 0"/>
+    <origin xyz="0 ${rack_t_setback} ${rack_t_elevation}" rpy="0 0 0"/>
   </xacro:rack_t>
   <!-- rack_b1 -->
@@ -42,6 +43,7 @@
     <origin xyz="${rack_width + rack_separation} 0 0" rpy="0 0 0"/>
   </xacro:rack_b>
+  <!-- rack_t1 -->
   <xacro:rack_t name="rack_t1" parent="rack_b1">
-    <origin xyz="0 0 ${rack_t_elevation}" rpy="0 0 0"/>
+    <origin xyz="0 ${rack_t_setback} ${rack_t_elevation}" rpy="0 0 0"/>
   </xacro:rack_t>
   <!-- rack_b2 -->
@@ -49,6 +51,7 @@
     <origin xyz="${rack_width + rack_separation} 0 0" rpy="0 0 0"/>
   </xacro:rack_b>
+  <!-- rack_t2 -->
   <xacro:rack_t name="rack_t2" parent="rack_b2">
-    <origin xyz="0 0 ${rack_t_elevation}" rpy="0 0 0"/>
+    <origin xyz="0 ${rack_t_setback} ${rack_t_elevation}" rpy="0 0 0"/>
   </xacro:rack_t>
   <!-- rack_b3 -->
@@ -56,14 +59,24 @@
     <origin xyz="${rack_width + rack_separation} 0 0" rpy="0 0 0"/>
   </xacro:rack_b>
+  <!-- rack_t3 -->
   <xacro:rack_t name="rack_t3" parent="rack_b3">
-    <origin xyz="0 0 ${rack_t_elevation}" rpy="0 0 0"/>
+    <origin xyz="0 ${rack_t_setback} ${rack_t_elevation}" rpy="0 0 0"/>
   </xacro:rack_t>
   <!-- rack_b4 -->
-  <xacro:rack_b name="rack_b4" parent="ground">
+  <xacro:rack_b name="rack_b4" parent="rack_b3">
+    <origin xyz="${rack_width + rack_separation} 0 0" rpy="0 0 0"/>
+  </xacro:rack_b>
+  <!-- rack_t4 -->
+  <xacro:rack_t name="rack_t4" parent="rack_b4">
+    <origin xyz="0 ${rack_t_setback} ${rack_t_elevation}" rpy="0 0 0"/>
+  </xacro:rack_t>
+  <!-- rack_b5 -->
+  <xacro:rack_b name="rack_b5" parent="ground">
     <origin xyz="${1.5 + rack_width} ${-workspace_length/2} 0"
 	    rpy="0 0 ${pi}"/>
   </xacro:rack_b>
-  <xacro:rack_t name="rack_t4" parent="rack_b4">
-    <origin xyz="0 0 ${rack_t_elevation}" rpy="0 0 0"/>
+  <!-- rack_t5 -->
+  <xacro:rack_t name="rack_t5" parent="rack_b5">
+    <origin xyz="0 ${rack_t_setback} ${rack_t_elevation}" rpy="0 0 0"/>
   </xacro:rack_t>
   <!-- Put boxes on shooters -->

File: nedo3_description/urdf/rack_b.urdf.xacro (robot description, xacro)
@@ -3,5 +3,5 @@
     <link name="${name}">
       <visual>
-        <origin rpy="0 0 0" xyz="0 0 0"/>
+        <origin xyz="0 0.050 0" rpy="0 0 0"/>
         <geometry>
           <mesh filename="package://nedo3_description/meshes/visual/rack_b.stl" scale="0.001 0.001 0.001"/>
@@ -12,5 +12,5 @@
       </visual>
       <collision>
-        <origin rpy="0 0 0" xyz="0 0.05 0"/>
+        <origin xyz="0 0.050 0" rpy="0 0 0"/>
         <geometry>
           <mesh filename="package://nedo3_description/meshes/collision/rack_b.stl" scale="0.001 0.001 0.001"/>

File: nedo3_description/urdf/rack_t.urdf.xacro (robot description, xacro)
@@ -3,5 +3,5 @@
     <link name="${name}">
       <visual>
-        <origin rpy="0 0 0" xyz="0 0 0"/>
+        <origin xyz="0 0 0" rpy="0 0 0"/>
         <geometry>
           <mesh filename="package://nedo3_description/meshes/visual/rack_t.stl" scale="0.001 0.001 0.001"/>
@@ -12,5 +12,5 @@
       </visual>
       <collision>
-        <origin rpy="0 0 0" xyz="0 0 0"/>
+        <origin xyz="0 0 0" rpy="0 0 0"/>
         <geometry>
           <mesh filename="package://nedo3_description/meshes/collision/rack_t.stl" scale="0.001 0.001 0.001"/>

Commit message: Add arm and gripper

File: nedo3_description/urdf/nedo3_demo.urdf.xacro (robot description, xacro)
@@ -1,4 +1,7 @@
 <?xml version="1.0"?>
 <robot xmlns:xacro="http://wiki.ros.org/xacro" name="showcase">
+  <xacro:arg name="kinematics_parameters_file"
+	     default="$(find ur_description
+		      )/config/ur5e/default_kinematics.yaml"/>
   <xacro:property name="lane_separation"	value="2.000"/>
   <xacro:property name="lane_width"		value="0.87"/>
@@ -9,4 +12,10 @@
   <xacro:property name="rack_t_setback"		value="-0.050"/>
   <xacro:property name="rack_t_elevation"	value="0.595"/>
+  <!-- UR5 physical installation (Tsukuba)-->
+  <xacro:property name="table_x" value="4.0"/>
+  <xacro:property name="table_y" value="-2.0"/>
+  <xacro:property name="table_w" value="0.3"/>
+  <xacro:property name="table_l" value="0.3"/>
+  <xacro:property name="table_h" value="0.7"/>
   <!-- Root frame -->
   <link name="world"/>
@@ -95,3 +104,40 @@
 			    part_props="${part_props}"
 			    box_props="${box_props}"/>
+  <!-- Table for mounting UR5e -->
+  <xacro:include filename="$(find nedo3_description)/urdf/table.urdf.xacro"/>
+  <xacro:table prefix="arm_"
+	       width="${table_w}" length="${table_l}" height="${table_h}"
+	       parent="ground">
+    <origin xyz="${table_x} ${table_y} 0" rpy="0 0 0"/>
+  </xacro:table>
+  <!-- Spawn UR5E arm -->
+  <xacro:include filename="$(find ur_gazebo)/urdf/ur_macro.xacro"/>
+  <xacro:ur_robot_gazebo
+      prefix="arm_"
+      joint_limits_parameters_file="$(find ur_description
+				    )/config/ur5e/joint_limits.yaml"
+      physical_parameters_file="$(find ur_description
+				)/config/ur5e/physical_parameters.yaml"
+      visual_parameters_file="$(find ur_description
+			      )/config/ur5e/visual_parameters.yaml"
+      kinematics_parameters_file="$(arg kinematics_parameters_file)"
+      transmission_hw_interface="hardware_interface/PositionJointInterface"/>
+  <joint name="arm_base_joint" type="fixed">
+    <origin xyz="${table_w/2} ${table_l/2} 0" rpy="0 0 0"/>
+    <parent link="arm_table_top" />
+    <child link="arm_base_link"/>
+  </joint>
+  <!-- Spawn and attach coupling -->
+  <xacro:include filename="$(find aist_robotiq
+  			   )/urdf/robotiq_arg2f_coupling.urdf.xacro"/>
+  <xacro:robotiq_arg2f_coupling prefix="gripper_coupling_" parent="arm_flange">
+    <origin xyz="0 0 0" rpy="0 0 0"/>
+  </xacro:robotiq_arg2f_coupling>
+  <!-- Spawn and attach gripper -->
+  <xacro:include filename="$(find aist_robotiq
+  			   )/urdf/robotiq_85_gripper.urdf.xacro"/>
+  <xacro:robotiq_85_gripper prefix="gripper_"
+			     parent="gripper_coupling_flange_link">
+    <origin xyz="0 0 0" rpy="0 0 0"/>
+  </xacro:robotiq_85_gripper>
 </robot>

Commit message: Fix orientation of gripper

File: nedo3_description/urdf/nedo3_demo.urdf.xacro (robot description, xacro)
@@ -124,6 +124,6 @@
       transmission_hw_interface="hardware_interface/PositionJointInterface"/>
   <joint name="arm_base_joint" type="fixed">
-    <origin xyz="${table_w/2} ${table_l/2} 0" rpy="0 0 0"/>
-    <parent link="arm_table_top" />
+    <origin xyz="0 0 0" rpy="0 0 0"/>
+    <parent link="arm_table_top_origin_center" />
     <child link="arm_base_link"/>
   </joint>
@@ -132,5 +132,5 @@
   			   )/urdf/robotiq_arg2f_coupling.urdf.xacro"/>
   <xacro:robotiq_arg2f_coupling prefix="gripper_coupling_" parent="arm_flange">
-    <origin xyz="0 0 0" rpy="0 0 0"/>
+    <origin xyz="0 0 0" rpy="${pi} 0 0"/>
   </xacro:robotiq_arg2f_coupling>
   <!-- Spawn and attach gripper -->

File: nedo3_moveit_config/config/gazebo_nedo3_demo.urdf (robot description, URDF)
Before this commit: robot nedo3_demo, 282 links, 281 joints
Joints:
- joint arm_base_joint: origin xyz=0.15 0.15 0 rpy=0 0 0 -> xyz=0 0 0 rpy=0 0 0; parent arm_table_top -> arm_table_top_origin_center
- joint gripper_coupling_base_joint: origin xyz=0 0 0 rpy=0 0 0 -> xyz=0 0 0 rpy=3.141592653589793 0 0

Commit message: Modify placement of rack and arm, and add urdf_publisher of dhaiba_ros

File: nedo3_description/urdf/nedo3_demo.urdf.xacro (robot description, xacro)
@@ -15,6 +15,6 @@
   <xacro:property name="table_x" value="4.0"/>
   <xacro:property name="table_y" value="-2.0"/>
-  <xacro:property name="table_w" value="0.3"/>
-  <xacro:property name="table_l" value="0.3"/>
+  <xacro:property name="table_w" value="1.0"/>
+  <xacro:property name="table_l" value="0.7"/>
   <xacro:property name="table_h" value="0.7"/>
   <!-- Root frame -->
@@ -82,5 +82,5 @@
   <!-- rack_b5 -->
   <xacro:rack_b name="rack_b5" parent="ground">
-    <origin xyz="${1.5 + rack_width} ${-workspace_length/2} 0"
+    <origin xyz="6.5 ${-workspace_length/2} 0"
 	    rpy="0 0 ${pi}"/>
   </xacro:rack_b>

File: nedo3_description/urdf/rack_b.urdf.xacro (robot description, xacro)
@@ -20,4 +20,5 @@
       <inertial>
 	<mass value="20.0"/>
+	<origin xyz="0.425 0.75 0.25" rpy="0 0 0"/>
 	<inertia ixx="0.0" ixy="0.0" ixz="0.0" iyy="0.0" iyz="0.0" izz="0.0"/>
       </inertial>

File: nedo3_description/urdf/rack_t.urdf.xacro (robot description, xacro)
@@ -20,4 +20,5 @@
       <inertial>
 	<mass value="20.0"/>
+	<origin xyz="0.425 0.75 0.4" rpy="0 0 0"/>
 	<inertia ixx="0.0" ixy="0.0" ixz="0.0" iyy="0.0" iyz="0.0" izz="0.0"/>
       </inertial>

File: nedo3_moveit_config/config/gazebo_nedo3_demo.urdf (robot description, URDF)
Before this commit: robot nedo3_demo, 282 links, 281 joints
Links:
- link arm_table_top: geometry collision box size=1.0 0.7 0.02; visual box size=1.0 0.7 0.02
Joints:
- joint arm_table_leg1: origin xyz=0.25 0 0 rpy=0 0 0 -> xyz=0.95 0 0 rpy=0 0 0
- joint arm_table_leg2: origin xyz=0 0.25 0 rpy=0 0 0 -> xyz=0 0.6499999999999999 0 rpy=0 0 0
- joint arm_table_leg3: origin xyz=0.25      0.25      0 rpy=0 0 0 -> xyz=0.95      0.6499999999999999      0 rpy=0 0 0
- joint arm_table_top_origin_center: origin xyz=0.15 0.15 0 rpy=0 0 0 -> xyz=0.5 0.35 0 rpy=0 0 0
- joint rack_b5_joint: origin xyz=2.35 -1.435 0 rpy=0 0 3.141592653589793 -> xyz=6.5 -1.435 0 rpy=0 0 3.141592653589793
