Commit message: Fix argument name representing YAML file for arm calibration

File: nedo3_moveit_config/config/gazebo_nedo3_demo.urdf (robot description, URDF)
Before this commit: robot nedo3_demo, 282 links, 281 joints
Links:
- removed link box_3
- removed link box_3_backside
- removed link box_3_bottom
- removed link box_3_center_bottom
- removed link box_3_center_top
- removed link box_3_frontside
- removed link box_3_leftside
- removed link box_3_lower_left_top
- removed link box_3_lower_right_top
- removed link box_3_rightside
- removed link box_3_upper_left_top
- removed link box_3_upper_right_top
- removed link box_4
- removed link box_4_backside
- removed link box_4_bottom
- removed link box_4_center_bottom
- removed link box_4_center_top
- removed link box_4_frontside
- removed link box_4_leftside
- removed link box_4_lower_left_top
- removed link box_4_lower_right_top
- removed link box_4_rightside
- removed link box_4_upper_left_top
- removed link box_4_upper_right_top
- link arm_base_link_inertia: geometry collision mesh filename=package://ur_description/meshes/ur5e/collision/base.stl; visual mesh filename=package://ur_description/meshes/ur5e/visual/base.stl
- link arm_forearm_link: geometry collision mesh filename=package://ur_description/meshes/ur5e/collision/forearm.stl; visual mesh filename=package://ur_description/meshes/ur5e/visual/forearm.stl
- link arm_shoulder_link: geometry collision mesh filename=package://ur_description/meshes/ur5e/collision/shoulder.stl; visual mesh filename=package://ur_description/meshes/ur5e/visual/shoulder.stl
- link arm_upper_arm_link: geometry collision mesh filename=package://ur_description/meshes/ur5e/collision/upperarm.stl; visual mesh filename=package://ur_description/meshes/ur5e/visual/upperarm.stl
- link arm_wrist_1_link: geometry collision mesh filename=package://ur_description/meshes/ur5e/collision/wrist1.stl; visual mesh filename=package://ur_description/meshes/ur5e/visual/wrist1.stl
- link arm_wrist_2_link: geometry collision mesh filename=package://ur_description/meshes/ur5e/collision/wrist2.stl; visual mesh filename=package://ur_description/meshes/ur5e/visual/wrist2.stl
- link arm_wrist_3_link: geometry collision mesh filename=package://ur_description/meshes/ur5e/collision/wrist3.stl; visual mesh filename=package://ur_description/meshes/ur5e/visual/wrist3.stl
Joints:
- removed joint box_3
- removed joint box_3_backside
- removed joint box_3_bottom_joint
- removed joint box_3_center_bottom_joint
- removed joint box_3_center_top_joint
- removed joint box_3_frontside
- removed joint box_3_leftside
- removed joint box_3_lower_left_top_joint
- removed joint box_3_lower_right_top_joint
- removed joint box_3_rightside
- removed joint box_3_upper_left_top_joint
- removed joint box_3_upper_right_top_joint
- removed joint box_4
- removed joint box_4_backside
- removed joint box_4_bottom_joint
- removed joint box_4_center_bottom_joint
- removed joint box_4_center_top_joint
- removed joint box_4_frontside
- removed joint box_4_leftside
- removed joint box_4_lower_left_top_joint
- removed joint box_4_lower_right_top_joint
- removed joint box_4_rightside
- removed joint box_4_upper_left_top_joint
- removed joint box_4_upper_right_top_joint
- joint box_5: parent rack_t2_lower -> rack_t5_lower
- joint box_9: parent rack_t2_lower -> rack_t5_lower
